Commit message: 第17天：URDF 两轮小车（joint + Xacro 宏 + 参数化 + 万向轮）

File: src/my_robot_description/urdf/my_robot.urdf.xacro (robot description, xacro)
@@ -1,9 +1,17 @@
 <?xml version="1.0"?>
 <robot name="my_robot" xmlns:xacro="http://www.ros.org/wiki/xacro">
+  <xacro:property name="wheel_radius" value="0.1"/>
+  <xacro:property name="wheel_width" value="0.04"/>
+  <xacro:property name="wheel_offset_y" value="0.2"/>
+  <xacro:property name="wheel_offset_z" value="${-base_height/2}"/>
+  <xacro:property name="base_length" value="0.6"/>
+  <xacro:property name="base_width" value="0.4"/>
+  <xacro:property name="base_height" value="0.2"/>
+  <xacro:property name="caster_radius" value="0.03"/>
   <link name="base_link">
     <visual>
       <origin xyz="0 0 0" rpy="0 0 0"/>
       <geometry>
-        <box size="3 3 3"/>
+        <box size="${base_length} ${base_width} ${base_height}"/>
       </geometry>
       <material name="blue">
@@ -14,5 +22,5 @@
       <origin xyz="0 0 0" rpy="0 0 0"/>
       <geometry>
-        <box size="3 3 3"/>
+        <box size="0.6 0.4 0.2"/>
       </geometry>
     </collision>
@@ -23,3 +31,66 @@
     </inertial>
   </link>
+  <xacro:macro name="caster" params="caster_name x_offset">
+    <link name="caster_${caster_name}">
+      <visual>
+        <origin xyz="0 0 0" rpy="0 0 0"/>
+        <geometry>
+          <sphere radius="${caster_radius}"/>
+        </geometry>
+        <material name="gray">
+          <color rgba="0.5 0.5 0.5 1.0"/>
+        </material>
+      </visual>
+      <collision>
+        <origin xyz="0 0 0" rpy="0 0 0"/>
+        <geometry>
+          <sphere radius="${caster_radius}"/>
+        </geometry>
+      </collision>
+      <inertial>
+        <origin xyz="0 0 0" rpy="0 0 0"/>
+        <mass value="0.1"/>
+        <inertia ixx="0.001" ixy="0" ixz="0" iyy="0.001" iyz="0" izz="0.001"/>
+      </inertial>
+    </link>
+    <joint name="caster_${caster_name}_joint" type="fixed">
+      <parent link="base_link"/>
+      <child  link="caster_${caster_name}"/>
+      <origin xyz="${x_offset} 0 ${wheel_offset_z}" rpy="0 0 0"/>
+    </joint>
+  </xacro:macro>
+  <xacro:caster caster_name="front" x_offset="0.25"/>
+  <xacro:caster caster_name="back"  x_offset="-0.25"/>
+  <xacro:macro name="wheel" params="wheel_name y_offset">
+    <link name="wheel_${wheel_name}">
+      <visual>
+        <origin xyz="0 0 0" rpy="0 0 0"/>
+        <geometry>
+          <cylinder radius="${wheel_radius}" length="${wheel_width}"/>
+        </geometry>
+        <material name="black">
+          <color rgba="0.1 0.1 0.1 1.0"/>
+        </material>
+      </visual>
+      <collision>
+        <origin xyz="0 0 0" rpy="0 0 0"/>
+        <geometry>
+          <cylinder radius="${wheel_radius}" length="${wheel_width}"/>
+        </geometry>
+      </collision>
+      <inertial>
+        <origin xyz="0 0 0" rpy="0 0 0"/>
+        <mass value="0.5"/>
+        <inertia ixx="0.001" ixy="0" ixz="0" iyy="0.001" iyz="0" izz="0.001"/>
+      </inertial>
+    </link>
+    <joint name="wheel_${wheel_name}_joint" type="continuous">
+      <parent link="base_link"/>
+      <child  link="wheel_${wheel_name}"/>
+      <origin xyz="0 ${y_offset} ${wheel_offset_z}" rpy="1.5708 0 0"/>
+      <axis xyz="0 0 1"/>
+    </joint>
+  </xacro:macro>
+  <xacro:wheel wheel_name="left"  y_offset="${wheel_offset_y}"/>
+  <xacro:wheel wheel_name="right" y_offset="${-wheel_offset_y}"/>
 </robot>

Commit message: 第18天：URDF 阶段四收尾（激光雷达 + 深度相机 + check_urdf 通过）

File: src/my_robot_description/urdf/my_robot.urdf.xacro (robot description, xacro)
@@ -1,12 +1,17 @@
 <?xml version="1.0"?>
 <robot name="my_robot" xmlns:xacro="http://www.ros.org/wiki/xacro">
+  <xacro:property name="base_length" value="0.6"/>
+  <xacro:property name="base_width" value="0.4"/>
+  <xacro:property name="base_height" value="0.2"/>
   <xacro:property name="wheel_radius" value="0.1"/>
   <xacro:property name="wheel_width" value="0.04"/>
   <xacro:property name="wheel_offset_y" value="0.2"/>
   <xacro:property name="wheel_offset_z" value="${-base_height/2}"/>
-  <xacro:property name="base_length" value="0.6"/>
-  <xacro:property name="base_width" value="0.4"/>
-  <xacro:property name="base_height" value="0.2"/>
   <xacro:property name="caster_radius" value="0.03"/>
+  <xacro:property name="laser_radius" value="0.05"/>
+  <xacro:property name="laser_height" value="0.04"/>
+  <xacro:property name="camera_size_x" value="0.02"/>
+  <xacro:property name="camera_size_y" value="0.08"/>
+  <xacro:property name="camera_size_z" value="0.08"/>
   <link name="base_link">
     <visual>
@@ -22,5 +27,5 @@
       <origin xyz="0 0 0" rpy="0 0 0"/>
       <geometry>
-        <box size="0.6 0.4 0.2"/>
+        <box size="${base_length} ${base_width} ${base_height}"/>
       </geometry>
     </collision>
@@ -92,4 +97,58 @@
     </joint>
   </xacro:macro>
+  <link name="laser_link">
+    <visual>
+      <origin xyz="0 0 0" rpy="0 0 0"/>
+      <geometry>
+        <cylinder radius="${laser_radius}" length="${laser_height}"/>
+      </geometry>
+      <material name="green">
+        <color rgba="0.1 0.5 0.1 1.0"/>
+      </material>
+    </visual>
+    <collision>
+      <origin xyz="0 0 0" rpy="0 0 0"/>
+      <geometry>
+        <cylinder radius="${laser_radius}" length="${laser_height}"/>
+      </geometry>
+    </collision>
+    <inertial>
+      <origin xyz="0 0 0" rpy="0 0 0"/>
+      <mass value="0.5"/>
+      <inertia ixx="0.001" ixy="0" ixz="0" iyy="0.001" iyz="0" izz="0.001"/>
+    </inertial>
+  </link>
+  <joint name="laser" type="fixed">
+    <parent link="base_link"/>
+    <child  link="laser_link"/>
+    <origin xyz="0 0 ${base_height/2 + laser_height/2}" rpy="0 0 0"/>
+  </joint>
+  <link name="camera_link">
+    <visual>
+      <origin xyz="0 0 0" rpy="0 0 0"/>
+      <geometry>
+         <box size="${camera_size_x} ${camera_size_y} ${camera_size_z}"/>
+      </geometry>
+      <material name="red">
+        <color rgba="0.5 0.1 0.1 1.0"/>
+      </material>
+    </visual>
+    <collision>
+      <origin xyz="0 0 0" rpy="0 0 0"/>
+      <geometry>
+        <box size="${camera_size_x} ${camera_size_y} ${camera_size_z}"/>
+      </geometry>
+    </collision>
+    <inertial>
+      <origin xyz="0 0 0" rpy="0 0 0"/>
+      <mass value="0.1"/>
+      <inertia ixx="0.001" ixy="0" ixz="0" iyy="0.001" iyz="0" izz="0.001"/>
+    </inertial>
+  </link>
+  <joint name="camera" type="fixed">
+    <parent link="base_link"/>
+    <child  link="camera_link"/>
+    <origin xyz="${base_length/2 + camera_size_x/2} 0 0" rpy="0 0 0"/>
+  </joint>
   <xacro:wheel wheel_name="left"  y_offset="${wheel_offset_y}"/>
   <xacro:wheel wheel_name="right" y_offset="${-wheel_offset_y}"/>

Commit message: Day22-23：Gazebo差速驱动+传感器；my_robot_description正式化；新增 10-原理与排查方法

File: src/my_robot_description/urdf/my_robot.urdf.xacro (robot description, xacro)
@@ -14,4 +14,5 @@
   <xacro:property name="camera_size_y" value="0.08"/>
   <xacro:property name="camera_size_z" value="0.08"/>
+  <xacro:property name="caster_offset_z" value="${wheel_offset_z - wheel_radius + caster_radius}"/>
     <!-- ① 摩擦（放前面，方便对照上面刚定义的轮子）-->
   <gazebo reference="wheel_left">
@@ -71,5 +72,5 @@
       <parent link="base_link"/>
       <child  link="caster_${caster_name}"/>
-      <origin xyz="${x_offset} 0 ${wheel_offset_z}" rpy="0 0 0"/>
+      <origin xyz="${x_offset} 0 ${caster_offset_z}" rpy="0 0 0"/>
     </joint>
   </xacro:macro>
@@ -106,4 +107,6 @@
     </joint>
   </xacro:macro>
+  <xacro:wheel wheel_name="left"  y_offset="${wheel_offset_y}"/>
+  <xacro:wheel wheel_name="right" y_offset="${-wheel_offset_y}"/>
   <link name="laser_link">
     <visual>
@@ -160,7 +163,5 @@
     <origin xyz="${base_length/2 + camera_size_x/2} 0 0" rpy="0 0 0"/>
   </joint>
-  <xacro:wheel wheel_name="left"  y_offset="${wheel_offset_y}"/>
-  <xacro:wheel wheel_name="right" y_offset="${-wheel_offset_y}"/>
-    <!-- ══════════ Gazebo 差速驱动 ══════════ -->
+    <!-- ══════════ Gazebo 差速驱动（插件） ══════════ -->
   <gazebo>
     <plugin filename="gz-sim-diff-drive-system"
@@ -178,3 +179,41 @@
     </plugin>
   </gazebo>
+    <!-- ══════════ 激光雷达传感器 ══════════ -->
+  <gazebo reference="base_link">
+    <sensor name="laser" type="gpu_lidar">
+      <gz_frame_id>laser_link</gz_frame_id>
+      <pose>0 0 0.5 0 0 0</pose>
+      <visualize>true</visualize>
+      <update_rate>10</update_rate>
+      <topic>scan</topic>
+      <always_on>1</always_on>
+      <lidar>
+        <scan>
+          <horizontal>
+            <samples>360</samples>
+            <resolution>1</resolution>
+            <min_angle>-3.14159</min_angle>
+            <max_angle>3.14159</max_angle>
+          </horizontal>
+        </scan>
+        <range>
+          <min>0.1</min>
+          <max>20.0</max>
+          <resolution>0.01</resolution>
+        </range>
+      </lidar>
+    </sensor>
+  </gazebo>
+  <gazebo>
+    <plugin filename="gz-sim-sensors-system"
+            name="gz::sim::systems::Sensors">
+      <render_engine>ogre2</render_engine>
+    </plugin>
+  </gazebo>
+  <gazebo>
+    <plugin filename="gz-sim-joint-state-publisher-system"
+            name="gz::sim::systems::JointStatePublisher">
+      <topic>/joint_states</topic>
+    </plugin>
+  </gazebo>
 </robot>
