Commit message: 第30-31天：ros2_control打通（包改名my_robot，新增坑82-84）；launch加可选RViz

File: src/my_robot/urdf/my_robot.urdf.xacro (robot description, xacro)
@@ -217,3 +217,27 @@
     </plugin>
   </gazebo>
+    <!-- ══════════ ros2_control（第 30 天的状态，先只声明）══════════ -->
+  <ros2_control name="GazeboSimSystem" type="system">
+    <hardware>
+      <plugin>gz_ros2_control/GazeboSimSystem</plugin>
+    </hardware>
+    <joint name="wheel_left_joint">
+      <command_interface name="velocity"/>
+      <state_interface name="position"/>
+      <state_interface name="velocity"/>
+    </joint>
+    <joint name="wheel_right_joint">
+      <command_interface name="velocity"/>
+      <state_interface name="position"/>
+      <state_interface name="velocity"/>
+    </joint>
+  </ros2_control>
+  <gazebo>
+    <plugin filename="gz_ros2_control-system" name="gz_ros2_control::GazeboSimROS2ControlPlugin">
+      <ros>
+        <namespace></namespace>
+      </ros>
+      <parameters>$(find my_robot)/config/ros2_control.yaml</parameters>
+    </plugin>
+  </gazebo>
 </robot>

Commit message: 第35-36天：定位并修复建图根因（轮子轴向反，坑95）；建图正确并保存 my_map_final；补坑 95-96

File: src/my_robot/urdf/my_robot.urdf.xacro (robot description, xacro)
@@ -104,5 +104,5 @@
       <child  link="wheel_${wheel_name}"/>
       <origin xyz="0 ${y_offset} ${wheel_offset_z}" rpy="1.5708 0 0"/>
-      <axis xyz="0 0 1"/>
+      <axis xyz="0 0 -1"/>
     </joint>
   </xacro:macro>
